Commit message: change ergo-jr to dragster-mini

File: software/poppy_dragster_mini/poppy-dragster-mini.urdf (robot description, URDF)
Before this commit: robot PoppyErgoJr, 7 links, 6 joints
Links:
- link base_link: geometry collision mesh filename=package://PoppyDragsterMini/meshes/base_link.STL; visual mesh filename=package://PoppyDragsterMini/meshes/base_link.STL
- link long_U: geometry collision mesh filename=package://PoppyDragsterMini/meshes/long_U.STL; visual mesh filename=package://PoppyDragsterMini/meshes/long_U.STL
- link section_1: geometry collision mesh filename=package://PoppyDragsterMini/meshes/section_1.STL; visual mesh filename=package://PoppyDragsterMini/meshes/section_1.STL
- link section_2: geometry collision mesh filename=package://PoppyDragsterMini/meshes/section_2.STL; visual mesh filename=package://PoppyDragsterMini/meshes/section_2.STL
- link section_3: geometry collision mesh filename=package://PoppyDragsterMini/meshes/section_3.STL; visual mesh filename=package://PoppyDragsterMini/meshes/section_3.STL
- link section_4: geometry collision mesh filename=package://PoppyDragsterMini/meshes/section_4.STL; visual mesh filename=package://PoppyDragsterMini/meshes/section_4.STL
- link tip: geometry collision mesh filename=package://PoppyDragsterMini/meshes/tip.STL; visual mesh filename=package://PoppyDragsterMini/meshes/tip.STL
